File: pcb/keyboard2.kicad_pcb (KiCad board)
At the start: 2 copper layers, 29 x 12 mm, 22 parts, among them J1 usb_pcb, J2 CONN_01X09, U1 atmega8u2-qfn, X1 resonator

Commit message: added and updated libraries
Parts:
- B1: footprint oscu_footprints:button_smd_panasonic -> keyboard2_footprints:button_smd_panasonic
- C1, C2, C3, C4: footprint oscu_footprints:C_0402_nosilk -> keyboard2_footprints:C_0402_nosilk
- D1, D2, D3, D4: footprint oscu_footprints:LED_0603_nosilk -> keyboard2_footprints:LED_0603_nosilk
- J1: footprint oscu_footprints:usb_pcb -> keyboard2_footprints:usb_pcb
- J2: footprint oscu_footprints:connector_smd_round2 -> keyboard2_footprints:connector_smd_round2
- R1, R2, R3, R4, R5, R6, R7: footprint oscu_footprints:R_0402_nosilk -> keyboard2_footprints:R_0402_nosilk
- U1: footprint oscu_footprints:qfn32_nosilk -> keyboard2_footprints:qfn32_nosilk
- X1: footprint oscu_footprints:resonator_murata_smd -> keyboard2_footprints:resonator_murata_smd
Changed lines of the file:
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@@
-(kicad_pcb (version 4) (host pcbnew "(after 2015-mar-04 BZR unknown)-product")
+(kicad_pcb (version 4) (host pcbnew 4.0.2-1.fc23-product)
   (general
     (links 50)
@@
   )
   (setup
-    (last_trace_width 0.2)
+    (last_trace_width 0.25)
     (user_trace_width 0.2)
     (trace_clearance 0.1)
@@
       (drillshape 0)
       (scaleselection 1)
-      (outputdirectory /home/oscu/Documents/Projects/KeyBoard/pcb2_plot/))
+      (outputdirectory ""))
   )
   (net 0 "")
@@
     (uvia_drill 0.1)
   )
-  (module oscu_footprints:usb_pcb (layer F.Cu)
+  (module keyboard2_footprints:usb_pcb (layer F.Cu)
     (at 167 109)
     (fp_text reference J1 (at 0 7) (layer F.SilkS) hide
@@
       (xy -9.920532 -1.897485) (xy -9.920356 -1.710484) (xy -9.920318 -1.50504) (xy -9.920318 -1.50504)) (layer F.SilkS) (width 0.1))
   )
-  (module oscu_footprints:R_0402_nosilk (layer F.Cu)
+  (module keyboard2_footprints:R_0402_nosilk (layer F.Cu)
     (at 157.75 113.25 270)
     (descr "Resistor SMD 0402, reflow soldering, Vishay (see dcrcw.pdf)")
@@
     )
   )
-  (module oscu_footprints:R_0402_nosilk (layer F.Cu)
+  (module keyboard2_footprints:R_0402_nosilk (layer F.Cu)
     (at 156.25 113.25 270)
     (descr "Resistor SMD 0402, reflow soldering, Vishay (see dcrcw.pdf)")
@@
     )
   )
-  (module oscu_footprints:R_0402_nosilk (layer F.Cu)
+  (module keyboard2_footprints:R_0402_nosilk (layer F.Cu)
     (at 157.75 104.75 90)
     (descr "Resistor SMD 0402, reflow soldering, Vishay (see dcrcw.pdf)")
@@
     )
   )
-  (module oscu_footprints:R_0402_nosilk (layer F.Cu)
+  (module keyboard2_footprints:R_0402_nosilk (layer F.Cu)
     (at 156.25 104.75 90)
     (descr "Resistor SMD 0402, reflow soldering, Vishay (see dcrcw.pdf)")
@@
     )
   )
-  (module oscu_footprints:R_0402_nosilk (layer F.Cu)
+  (module keyboard2_footprints:R_0402_nosilk (layer F.Cu)
     (at 163 108.5 180)
     (descr "Resistor SMD 0402, reflow soldering, Vishay (see dcrcw.pdf)")
@@
     )
   )
-  (module oscu_footprints:R_0402_nosilk (layer F.Cu)
+  (module keyboard2_footprints:R_0402_nosilk (layer F.Cu)
     (at 163 110 180)
     (descr "Resistor SMD 0402, reflow soldering, Vishay (see dcrcw.pdf)")
@@
     )
   )
-  (module oscu_footprints:button_smd_panasonic (layer F.Cu)
+  (module keyboard2_footprints:button_smd_panasonic (layer F.Cu)
     (at 152.25 109 180)
     (fp_text reference B1 (at 0 3.75 180) (layer F.SilkS) hide
@@
       (net 12 GND))
   )
-  (module oscu_footprints:resonator_murata_smd (layer F.Cu)
+  (module keyboard2_footprints:resonator_murata_smd (layer F.Cu)
     (at 162 104.75 180)
     (fp_text reference X1 (at 0 2 180) (layer F.SilkS) hide
@@
       (net 2 "Net-(U1-Pad2)"))
   )
-  (module oscu_footprints:LED_0603_nosilk (layer F.Cu)
+  (module keyboard2_footprints:LED_0603_nosilk (layer F.Cu)
     (at 150.25 104.75 180)
     (descr "LED 0603 smd package")
@@
       (net 12 GND))
   )
-  (module oscu_footprints:LED_0603_nosilk (layer F.Cu)
+  (module keyboard2_footprints:LED_0603_nosilk (layer F.Cu)
     (at 154 104.75 180)
     (descr "LED 0603 smd package")
@@
       (net 12 GND))
   )
-  (module oscu_footprints:LED_0603_nosilk (layer F.Cu)
+  (module keyboard2_footprints:LED_0603_nosilk (layer F.Cu)
     (at 150.25 113.25 180)
     (descr "LED 0603 smd package")
@@
       (net 12 GND))
   )
-  (module oscu_footprints:LED_0603_nosilk (layer F.Cu)
+  (module keyboard2_footprints:LED_0603_nosilk (layer F.Cu)
     (at 154 113.25 180)
     (descr "LED 0603 smd package")
@@
       (net 12 GND))
   )
-  (module oscu_footprints:connector_smd_round2 (layer B.Cu)
+  (module keyboard2_footprints:connector_smd_round2 (layer B.Cu)
     (at 155 109)
     (fp_text reference J2 (at 0 -7) (layer B.SilkS) hide
@@
       (net 19 /RXD))
   )
-  (module oscu_footprints:qfn32_nosilk (layer F.Cu)
+  (module keyboard2_footprints:qfn32_nosilk (layer F.Cu)
     (at 158.75 109 270)
     (fp_text reference U1 (at 0 -3.75 270) (layer F.SilkS) hide
@@
       (xy 2.817833 4.548849)) (layer B.SilkS) (width 0.1))
   )
-  (module oscu_footprints:C_0402_nosilk (layer F.Cu)
+  (module keyboard2_footprints:C_0402_nosilk (layer F.Cu)
     (at 163 111.5)
     (descr "Resistor SMD 0402, reflow soldering, Vishay (see dcrcw.pdf)")
@@
     )
   )
-  (module oscu_footprints:C_0402_nosilk (layer F.Cu)
+  (module keyboard2_footprints:C_0402_nosilk (layer F.Cu)
     (at 159.25 104.75 90)
     (descr "Resistor SMD 0402, reflow soldering, Vishay (see dcrcw.pdf)")
@@
     )
   )
-  (module oscu_footprints:C_0402_nosilk (layer F.Cu)
+  (module keyboard2_footprints:C_0402_nosilk (layer F.Cu)
     (at 163 107)
     (descr "Resistor SMD 0402, reflow soldering, Vishay (see dcrcw.pdf)")
@@
     )
   )
-  (module oscu_footprints:C_0402_nosilk (layer F.Cu)
+  (module keyboard2_footprints:C_0402_nosilk (layer F.Cu)
     (at 159.25 113.25 270)
     (descr "Resistor SMD 0402, reflow soldering, Vishay (see dcrcw.pdf)")
@@
     )
   )
-  (module oscu_footprints:R_0402_nosilk (layer F.Cu)
+  (module keyboard2_footprints:R_0402_nosilk (layer F.Cu)
     (at 160.75 113.25 270)
     (descr "Resistor SMD 0402, reflow soldering, Vishay (see dcrcw.pdf)")

Commit message: update reset capacitor not mounted
Parts:
- C1, C2, C3: value C -> 1u
- C4: value C -> not mounted
- D1: value led1 -> led_red
- D2: value led1 -> led_green
- D3: value led1 -> led_blue
- D4: value led1 -> led_yellow
- R1, R2: value R -> 22
- R3, R4, R6: value R -> 270
- R5: value R -> 1k
- R7: value R -> 4k7
Connections:
- U1 pad 11: (no net) -> Net-(U1-Pad11)
- U1 pad 12: (no net) -> Net-(U1-Pad12)
- U1 pad 13: (no net) -> Net-(U1-Pad13)
- U1 pad 14: (no net) -> Net-(U1-Pad14)
- U1 pad 20: (no net) -> Net-(U1-Pad20)
- U1 pad 21: (no net) -> Net-(U1-Pad21)
- U1 pad 22: (no net) -> Net-(U1-Pad22)
- U1 pad 23: (no net) -> Net-(U1-Pad23)
- U1 pad 25: (no net) -> Net-(U1-Pad25)
- U1 pad 26: (no net) -> Net-(U1-Pad26)
- U1 pad 5: (no net) -> Net-(U1-Pad5)
Changed lines of the file:
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@@
     (links 50)
     (no_connects 0)
-    (area 131.964287 91.9 185.75 123.050001)
+    (area 143.949999 102.949999 173.050001 115.050001)
     (thickness 1.6)
     (drawings 32)
@@
     (zones 0)
     (modules 22)
-    (nets 25)
+    (nets 36)
   )
   (page A4)
@@
   (net 23 "Net-(R5-Pad1)")
   (net 24 "Net-(R6-Pad1)")
+  (net 25 "Net-(U1-Pad11)")
+  (net 26 "Net-(U1-Pad12)")
+  (net 27 "Net-(U1-Pad13)")
+  (net 28 "Net-(U1-Pad14)")
+  (net 29 "Net-(U1-Pad25)")
+  (net 30 "Net-(U1-Pad26)")
+  (net 31 "Net-(U1-Pad20)")
+  (net 32 "Net-(U1-Pad21)")
+  (net 33 "Net-(U1-Pad22)")
+  (net 34 "Net-(U1-Pad23)")
+  (net 35 "Net-(U1-Pad5)")
   (net_class Default "This is the default net class."
     (clearance 0.1)
@@
     (add_net "Net-(R6-Pad1)")
     (add_net "Net-(U1-Pad1)")
+    (add_net "Net-(U1-Pad11)")
+    (add_net "Net-(U1-Pad12)")
+    (add_net "Net-(U1-Pad13)")
+    (add_net "Net-(U1-Pad14)")
     (add_net "Net-(U1-Pad2)")
+    (add_net "Net-(U1-Pad20)")
+    (add_net "Net-(U1-Pad21)")
+    (add_net "Net-(U1-Pad22)")
+    (add_net "Net-(U1-Pad23)")
+    (add_net "Net-(U1-Pad25)")
+    (add_net "Net-(U1-Pad26)")
+    (add_net "Net-(U1-Pad5)")
   )
   (net_class thin ""
@@
       (effects (font (size 1 1) (thickness 0.15)))
     )
-    (fp_text value R (at 0 1.8 270) (layer F.Fab)
+    (fp_text value 270 (at 0 1.8 270) (layer F.Fab)
       (effects (font (size 1 1) (thickness 0.15)))
     )
@@
       (effects (font (size 1 1) (thickness 0.15)))
     )
-    (fp_text value R (at 0 1.8 270) (layer F.Fab)
+    (fp_text value 1k (at 0 1.8 270) (layer F.Fab)
       (effects (font (size 1 1) (thickness 0.15)))
     )
@@
       (effects (font (size 1 1) (thickness 0.15)))
     )
-    (fp_text value R (at 0 1.8 90) (layer F.Fab)
+    (fp_text value 270 (at 0 1.8 90) (layer F.Fab)
       (effects (font (size 1 1) (thickness 0.15)))
     )
@@
       (effects (font (size 1 1) (thickness 0.15)))
     )
-    (fp_text value R (at 0 1.8 90) (layer F.Fab)
+    (fp_text value 270 (at 0 1.8 90) (layer F.Fab)
       (effects (font (size 1 1) (thickness 0.15)))
     )
@@
       (effects (font (size 1 1) (thickness 0.15)))
     )
-    (fp_text value R (at 0 1.8 180) (layer F.Fab)
+    (fp_text value 22 (at 0 1.8 180) (layer F.Fab)
       (effects (font (size 1 1) (thickness 0.15)))
     )
@@
       (effects (font (size 1 1) (thickness 0.15)))
     )
-    (fp_text value R (at 0 1.8 180) (layer F.Fab)
+    (fp_text value 22 (at 0 1.8 180) (layer F.Fab)
       (effects (font (size 1 1) (thickness 0.15)))
     )
@@
       (effects (font (size 1 1) (thickness 0.15)))
     )
-    (fp_text value led1 (at 0 1.016 180) (layer F.Fab)
+    (fp_text value led_red (at 0 1.016 180) (layer F.Fab)
       (effects (font (size 1 1) (thickness 0.15)))
     )
@@
       (effects (font (size 1 1) (thickness 0.15)))
     )
-    (fp_text value led1 (at 0 1.016 180) (layer F.Fab)
+    (fp_text value led_green (at 0 1.016 180) (layer F.Fab)
       (effects (font (size 1 1) (thickness 0.15)))
     )
@@
       (effects (font (size 1 1) (thickness 0.15)))
     )
-    (fp_text value led1 (at 0 1.016 180) (layer F.Fab)
+    (fp_text value led_blue (at 0 1.016 180) (layer F.Fab)
       (effects (font (size 1 1) (thickness 0.15)))
     )
@@
       (effects (font (size 1 1) (thickness 0.15)))
     )
-    (fp_text value led1 (at 0 1.016 180) (layer F.Fab)
+    (fp_text value led_yellow (at 0 1.016 180) (layer F.Fab)
       (effects (font (size 1 1) (thickness 0.15)))
     )
@@
     (pad 10 smd oval (at -1.25 2.5) (size 0.8 0.3) (layers F.Cu F.Paste F.Mask)
       (net 11 "Net-(B1-Pad3)"))
-    (pad 11 smd oval (at -0.75 2.5) (size 0.8 0.3) (layers F.Cu F.Paste F.Mask))
-    (pad 12 smd oval (at -0.25 2.5) (size 0.8 0.3) (layers F.Cu F.Paste F.Mask))
-    (pad 13 smd oval (at 0.25 2.5) (size 0.8 0.3) (layers F.Cu F.Paste F.Mask))
-    (pad 14 smd oval (at 0.75 2.5) (size 0.8 0.3) (layers F.Cu F.Paste F.Mask))
+    (pad 11 smd oval (at -0.75 2.5) (size 0.8 0.3) (layers F.Cu F.Paste F.Mask)
+      (net 25 "Net-(U1-Pad11)"))
+    (pad 12 smd oval (at -0.25 2.5) (size 0.8 0.3) (layers F.Cu F.Paste F.Mask)
+      (net 26 "Net-(U1-Pad12)"))
+    (pad 13 smd oval (at 0.25 2.5) (size 0.8 0.3) (layers F.Cu F.Paste F.Mask)
+      (net 27 "Net-(U1-Pad13)"))
+    (pad 14 smd oval (at 0.75 2.5) (size 0.8 0.3) (layers F.Cu F.Paste F.Mask)
+      (net 28 "Net-(U1-Pad14)"))
     (pad 15 smd oval (at 1.25 2.5) (size 0.8 0.3) (layers F.Cu F.Paste F.Mask)
       (net 14 /SCLK))
     (pad 16 smd oval (at 1.75 2.5) (size 0.8 0.3) (layers F.Cu F.Paste F.Mask)
       (net 15 /MOSI))
-    (pad 25 smd oval (at 1.75 -2.5) (size 0.8 0.3) (layers F.Cu F.Paste F.Mask))
-    (pad 26 smd oval (at 1.25 -2.5) (size 0.8 0.3) (layers F.Cu F.Paste F.Mask))
+    (pad 25 smd oval (at 1.75 -2.5) (size 0.8 0.3) (layers F.Cu F.Paste F.Mask)
+      (net 29 "Net-(U1-Pad25)"))
+    (pad 26 smd oval (at 1.25 -2.5) (size 0.8 0.3) (layers F.Cu F.Paste F.Mask)
+      (net 30 "Net-(U1-Pad26)"))
     (pad 27 smd oval (at 0.75 -2.5) (size 0.8 0.3) (layers F.Cu F.Paste F.Mask)
       (net 18 "Net-(C1-Pad1)"))
@@
     (pad 19 smd oval (at 2.5 0.75 270) (size 0.8 0.3) (layers F.Cu F.Paste F.Mask)
       (net 24 "Net-(R6-Pad1)"))
-    (pad 20 smd oval (at 2.5 0.25 270) (size 0.8 0.3) (layers F.Cu F.Paste F.Mask))
-    (pad 21 smd oval (at 2.5 -0.25 270) (size 0.8 0.3) (layers F.Cu F.Paste F.Mask))
-    (pad 22 smd oval (at 2.5 -0.75 270) (size 0.8 0.3) (layers F.Cu F.Paste F.Mask))
-    (pad 23 smd oval (at 2.5 -1.25 270) (size 0.8 0.3) (layers F.Cu F.Paste F.Mask))
+    (pad 20 smd oval (at 2.5 0.25 270) (size 0.8 0.3) (layers F.Cu F.Paste F.Mask)
+      (net 31 "Net-(U1-Pad20)"))
+    (pad 21 smd oval (at 2.5 -0.25 270) (size 0.8 0.3) (layers F.Cu F.Paste F.Mask)
+      (net 32 "Net-(U1-Pad21)"))
+    (pad 22 smd oval (at 2.5 -0.75 270) (size 0.8 0.3) (layers F.Cu F.Paste F.Mask)
+      (net 33 "Net-(U1-Pad22)"))
+    (pad 23 smd oval (at 2.5 -1.25 270) (size 0.8 0.3) (layers F.Cu F.Paste F.Mask)
+      (net 34 "Net-(U1-Pad23)"))
     (pad 24 smd oval (at 2.5 -1.75 270) (size 0.8 0.3) (layers F.Cu F.Paste F.Mask)
       (net 17 /RESET))
@@
     (pad 4 smd oval (at -2.5 -0.25 270) (size 0.8 0.3) (layers F.Cu F.Paste F.Mask)
       (net 13 +5V))
-    (pad 5 smd oval (at -2.5 0.25 270) (size 0.8 0.3) (layers F.Cu F.Paste F.Mask))
+    (pad 5 smd oval (at -2.5 0.25 270) (size 0.8 0.3) (layers F.Cu F.Paste F.Mask)
+      (net 35 "Net-(U1-Pad5)"))
     (pad 6 smd oval (at -2.5 0.75 270) (size 0.8 0.3) (layers F.Cu F.Paste F.Mask)
       (net 22 "Net-(R4-Pad1)"))
@@
       (effects (font (size 1 1) (thickness 0.15)))
     )
-    (fp_text value C (at 0 1.8) (layer F.Fab)
+    (fp_text value 1u (at 0 1.8) (layer F.Fab)
       (effects (font (size 1 1) (thickness 0.15)))
     )
@@
       (effects (font (size 1 1) (thickness 0.15)))
     )
-    (fp_text value C (at 0 1.8 90) (layer F.Fab)
+    (fp_text value 1u (at 0 1.8 90) (layer F.Fab)
       (effects (font (size 1 1) (thickness 0.15)))
     )
@@
       (effects (font (size 1 1) (thickness 0.15)))
     )
-    (fp_text value C (at 0 1.8) (layer F.Fab)
+    (fp_text value 1u (at 0 1.8) (layer F.Fab)
       (effects (font (size 1 1) (thickness 0.15)))
     )
@@
       (effects (font (size 1 1) (thickness 0.15)))
     )
-    (fp_text value C (at 0 1.8 270) (layer F.Fab)
+    (fp_text value "not mounted" (at 0 1.8 270) (layer F.Fab)
       (effects (font (size 1 1) (thickness 0.15)))
     )
@@
       (effects (font (size 1 1) (thickness 0.15)))
     )
-    (fp_text value R (at 0 1.8 270) (layer F.Fab)
-      (effects (font (size 1 1) (thickness 0.15)))
-    )
+    (fp_text value 4k7 (at 0 1.8 270) (layer F.Fab)
+      (effects (font (size 1 1) (thickness 0.15)))
+    )
